File: pcb/StopLight4/StopLight4.sch (KiCad schematic (older format))
At the start: 62 parts, among them J1 1935336, J2 1935336, J3 Remote Header, Q1 BT136-600, Q2 BT136-600, Q3 BT136-600, Q5 2N3904, T1 FS20-600, U1 L7805, U10 MOC3021M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

Commit message: Smaller PCB, sent to production!
Parts:
- removed F1, F2, F3: Fuse, Fuse:Fuseholder_Cylinder-6.3x32mm_Schurter_0031-8002_Horizontal_Open, symbol Device:Fuse
- J1, J2: footprint StopLight1:1935336 -> StopLight4:1984633
- R10, R20, R31: value 220 -> 220R; footprint Resistor_THT:R_Axial_DIN0207_L6.3mm_D2.5mm_P7.62mm_Horizontal -> Resistor_THT:R_Axial_DIN0207_L6.3mm_D2.5mm_P10.16mm_Horizontal
- R11, R12, R13, R14, R21, R22, R23, R24, R30, R32, R33, R34, R4, R5, R6, R7: footprint Resistor_THT:R_Axial_DIN0207_L6.3mm_D2.5mm_P7.62mm_Horizontal -> Resistor_THT:R_Axial_DIN0207_L6.3mm_D2.5mm_P10.16mm_Horizontal
Connections:
- net at J2.2: now also Q2.2 (A2), R24.1
- net at J2.3: now also Q3.2 (A2), R34.1
- net at J2.1: now also Q1.2 (A2), R14.1
Changed lines of the file:
@@
-$EndComp
-$Comp
-L Device:Fuse F2
-U 1 1 5F3C6F25
-P 8400 2700
-F 0 "F2" V 8300 2600 50  0000 L CNN
-F 1 "Fuse" V 8200 2600 50  0000 L CNN
-F 2 "Fuse:Fuseholder_Cylinder-6.3x32mm_Schurter_0031-8002_Horizontal_Open" V 8330 2700 50  0001 C CNN
-F 3 "~" H 8400 2700 50  0001 C CNN
-	1    8400 2700
-	0    1    1    0
 $EndComp
 $Comp
@@
 F 3 "~" H 950 1150 50  0001 C CNN
 	1    950  1150
-	0    1    1    0
-$EndComp
-$Comp
-L Device:Fuse F1
-U 1 1 5F3C87EA
-P 8400 1650
-F 0 "F1" V 8300 1550 50  0000 L CNN
-F 1 "Fuse" V 8200 1550 50  0000 L CNN
-F 2 "Fuse:Fuseholder_Cylinder-6.3x32mm_Schurter_0031-8002_Horizontal_Open" V 8330 1650 50  0001 C CNN
-F 3 "~" H 8400 1650 50  0001 C CNN
-	1    8400 1650
 	0    1    1    0
 $EndComp
@@
 F 0 "R11" V 4795 4000 50  0000 C CNN
 F 1 "220R" V 4886 4000 50  0000 C CNN
-F 2 "Resistor_THT:R_Axial_DIN0207_L6.3mm_D2.5mm_P7.62mm_Horizontal" H 5000 4000 50  0001 C CNN
+F 2 "Resistor_THT:R_Axial_DIN0207_L6.3mm_D2.5mm_P10.16mm_Horizontal" H 5000 4000 50  0001 C CNN
 F 3 "~" H 5000 4000 50  0001 C CNN
 	1    5000 4000
@@
 P 5000 4600
 F 0 "R31" V 4795 4600 50  0000 C CNN
-F 1 "220" V 4886 4600 50  0000 C CNN
-F 2 "Resistor_THT:R_Axial_DIN0207_L6.3mm_D2.5mm_P7.62mm_Horizontal" H 5000 4600 50  0001 C CNN
+F 1 "220R" V 4886 4600 50  0000 C CNN
+F 2 "Resistor_THT:R_Axial_DIN0207_L6.3mm_D2.5mm_P10.16mm_Horizontal" H 5000 4600 50  0001 C CNN
 F 3 "~" H 5000 4600 50  0001 C CNN
 	1    5000 4600
@@
 F 0 "R5" V 5245 1300 50  0000 C CNN
 F 1 "220R" V 5336 1300 50  0000 C CNN
-F 2 "Resistor_THT:R_Axial_DIN0207_L6.3mm_D2.5mm_P7.62mm_Horizontal" H 5450 1300 50  0001 C CNN
+F 2 "Resistor_THT:R_Axial_DIN0207_L6.3mm_D2.5mm_P10.16mm_Horizontal" H 5450 1300 50  0001 C CNN
 F 3 "~" H 5450 1300 50  0001 C CNN
 	1    5450 1300
@@
 F 0 "J1" H 2828 5453 60  0000 L CNN
 F 1 "1935336" H 2828 5347 60  0000 L CNN
-F 2 "StopLight1:1935336" H 2700 5290 60  0001 C CNN
+F 2 "StopLight4:1984633" H 2700 5290 60  0001 C CNN
 F 3 "" H 2300 5550 60  0000 C CNN
 	1    2300 5550
@@
 F 0 "R13" V 6743 2100 50  0000 C CNN
 F 1 "390R" V 6834 2100 50  0000 C CNN
-F 2 "Resistor_THT:R_Axial_DIN0207_L6.3mm_D2.5mm_P7.62mm_Horizontal" V 6880 2100 50  0001 C CNN
+F 2 "Resistor_THT:R_Axial_DIN0207_L6.3mm_D2.5mm_P10.16mm_Horizontal" V 6880 2100 50  0001 C CNN
 F 3 "~" H 6950 2100 50  0001 C CNN
 	1    6950 2100
@@
 F 0 "R14" V 7243 1650 50  0000 C CNN
 F 1 "51R" V 7334 1650 50  0000 C CNN
-F 2 "Resistor_THT:R_Axial_DIN0207_L6.3mm_D2.5mm_P7.62mm_Horizontal" V 7380 1650 50  0001 C CNN
+F 2 "Resistor_THT:R_Axial_DIN0207_L6.3mm_D2.5mm_P10.16mm_Horizontal" V 7380 1650 50  0001 C CNN
 F 3 "~" H 7450 1650 50  0001 C CNN
 	1    7450 1650
@@
 F 0 "R12" V 6743 1650 50  0000 C CNN
 F 1 "150R" V 6834 1650 50  0000 C CNN
-F 2 "Resistor_THT:R_Axial_DIN0207_L6.3mm_D2.5mm_P7.62mm_Horizontal" V 6880 1650 50  0001 C CNN
+F 2 "Resistor_THT:R_Axial_DIN0207_L6.3mm_D2.5mm_P10.16mm_Horizontal" V 6880 1650 50  0001 C CNN
 F 3 "~" H 6950 1650 50  0001 C CNN
 	1    6950 1650
@@
 F 0 "R23" V 6743 3150 50  0000 C CNN
 F 1 "390R" V 6834 3150 50  0000 C CNN
-F 2 "Resistor_THT:R_Axial_DIN0207_L6.3mm_D2.5mm_P7.62mm_Horizontal" V 6880 3150 50  0001 C CNN
+F 2 "Resistor_THT:R_Axial_DIN0207_L6.3mm_D2.5mm_P10.16mm_Horizontal" V 6880 3150 50  0001 C CNN
 F 3 "~" H 6950 3150 50  0001 C CNN
 	1    6950 3150
@@
 F 0 "R24" V 7243 2700 50  0000 C CNN
 F 1 "51R" V 7334 2700 50  0000 C CNN
-F 2 "Resistor_THT:R_Axial_DIN0207_L6.3mm_D2.5mm_P7.62mm_Horizontal" V 7380 2700 50  0001 C CNN
+F 2 "Resistor_THT:R_Axial_DIN0207_L6.3mm_D2.5mm_P10.16mm_Horizontal" V 7380 2700 50  0001 C CNN
 F 3 "~" H 7450 2700 50  0001 C CNN
 	1    7450 2700
@@
 F 0 "R22" V 6743 2700 50  0000 C CNN
 F 1 "150R" V 6834 2700 50  0000 C CNN
-F 2 "Resistor_THT:R_Axial_DIN0207_L6.3mm_D2.5mm_P7.62mm_Horizontal" V 6880 2700 50  0001 C CNN
+F 2 "Resistor_THT:R_Axial_DIN0207_L6.3mm_D2.5mm_P10.16mm_Horizontal" V 6880 2700 50  0001 C CNN
 F 3 "~" H 6950 2700 50  0001 C CNN
 	1    6950 2700
@@
 P 5500 3150
 F 0 "R20" V 5295 3150 50  0000 C CNN
-F 1 "220" V 5386 3150 50  0000 C CNN
-F 2 "Resistor_THT:R_Axial_DIN0207_L6.3mm_D2.5mm_P7.62mm_Horizontal" H 5500 3150 50  0001 C CNN
+F 1 "220R" V 5386 3150 50  0000 C CNN
+F 2 "Resistor_THT:R_Axial_DIN0207_L6.3mm_D2.5mm_P10.16mm_Horizontal" H 5500 3150 50  0001 C CNN
 F 3 "~" H 5500 3150 50  0001 C CNN
 	1    5500 3150
@@
 F 0 "R33" V 6693 4950 50  0000 C CNN
 F 1 "390R" V 6784 4950 50  0000 C CNN
-F 2 "Resistor_THT:R_Axial_DIN0207_L6.3mm_D2.5mm_P7.62mm_Horizontal" V 6830 4950 50  0001 C CNN
+F 2 "Resistor_THT:R_Axial_DIN0207_L6.3mm_D2.5mm_P10.16mm_Horizontal" V 6830 4950 50  0001 C CNN
 F 3 "~" H 6900 4950 50  0001 C CNN
 	1    6900 4950
@@
 F 0 "R34" V 7193 4500 50  0000 C CNN
 F 1 "51R" V 7284 4500 50  0000 C CNN
-F 2 "Resistor_THT:R_Axial_DIN0207_L6.3mm_D2.5mm_P7.62mm_Horizontal" V 7330 4500 50  0001 C CNN
+F 2 "Resistor_THT:R_Axial_DIN0207_L6.3mm_D2.5mm_P10.16mm_Horizontal" V 7330 4500 50  0001 C CNN
 F 3 "~" H 7400 4500 50  0001 C CNN
 	1    7400 4500
@@
 F 0 "R32" V 6693 4500 50  0000 C CNN
 F 1 "150R" V 6784 4500 50  0000 C CNN
-F 2 "Resistor_THT:R_Axial_DIN0207_L6.3mm_D2.5mm_P7.62mm_Horizontal" V 6830 4500 50  0001 C CNN
+F 2 "Resistor_THT:R_Axial_DIN0207_L6.3mm_D2.5mm_P10.16mm_Horizontal" V 6830 4500 50  0001 C CNN
 F 3 "~" H 6900 4500 50  0001 C CNN
 	1    6900 4500
@@
 F 0 "R30" V 5295 4950 50  0000 C CNN
 F 1 "220R" V 5386 4950 50  0000 C CNN
-F 2 "Resistor_THT:R_Axial_DIN0207_L6.3mm_D2.5mm_P7.62mm_Horizontal" H 5500 4950 50  0001 C CNN
+F 2 "Resistor_THT:R_Axial_DIN0207_L6.3mm_D2.5mm_P10.16mm_Horizontal" H 5500 4950 50  0001 C CNN
 F 3 "~" H 5500 4950 50  0001 C CNN
 	1    5500 4950
@@
 P 5500 2100
 F 0 "R10" V 5295 2100 50  0000 C CNN
-F 1 "220" V 5386 2100 50  0000 C CNN
-F 2 "Resistor_THT:R_Axial_DIN0207_L6.3mm_D2.5mm_P7.62mm_Horizontal" H 5500 2100 50  0001 C CNN
+F 1 "220R" V 5386 2100 50  0000 C CNN
+F 2 "Resistor_THT:R_Axial_DIN0207_L6.3mm_D2.5mm_P10.16mm_Horizontal" H 5500 2100 50  0001 C CNN
 F 3 "~" H 5500 2100 50  0001 C CNN
 	1    5500 2100
@@
 F 0 "R21" V 4795 4400 50  0000 C CNN
 F 1 "220R" V 4886 4400 50  0000 C CNN
-F 2 "Resistor_THT:R_Axial_DIN0207_L6.3mm_D2.5mm_P7.62mm_Horizontal" H 5000 4400 50  0001 C CNN
+F 2 "Resistor_THT:R_Axial_DIN0207_L6.3mm_D2.5mm_P10.16mm_Horizontal" H 5000 4400 50  0001 C CNN
 F 3 "~" H 5000 4400 50  0001 C CNN
 	1    5000 4400
@@
 Wire Wire Line
 	7500 4500 7700 4500
-$Comp
-L Device:Fuse F3
-U 1 1 5F3C807B
-P 8350 4500
-F 0 "F3" V 8250 4400 50  0000 L CNN
-F 1 "Fuse" V 8150 4400 50  0000 L CNN
-F 2 "Fuse:Fuseholder_Cylinder-6.3x32mm_Schurter_0031-8002_Horizontal_Open" V 8280 4500 50  0001 C CNN
-F 3 "~" H 8350 4500 50  0001 C CNN
-	1    8350 4500
-	0    1    1    0
-$EndComp
-Wire Wire Line
-	7750 2700 8250 2700
-Wire Wire Line
-	7750 1650 8250 1650
-Wire Wire Line
-	8200 4500 7700 4500
 Wire Wire Line
 	7200 3150 7750 3150
@@
 Wire Wire Line
 	9200 2700 9200 2200
-Wire Wire Line
-	8550 2700 9200 2700
 Wire Wire Line
 	9450 1350 9450 2400
@@
 F 0 "J2" H 10078 2003 60  0000 L CNN
 F 1 "1935336" H 10078 1897 60  0000 L CNN
-F 2 "StopLight1:1935336" H 9950 1840 60  0001 C CNN
+F 2 "StopLight4:1984633" H 9950 1840 60  0001 C CNN
 F 3 "" H 9550 2100 60  0000 C CNN
 	1    9550 2100
@@
 F 0 "R6" V 6195 3800 50  0000 C CNN
 F 1 "220R" V 6286 3800 50  0000 C CNN
-F 2 "Resistor_THT:R_Axial_DIN0207_L6.3mm_D2.5mm_P7.62mm_Horizontal" H 6400 3800 50  0001 C CNN
+F 2 "Resistor_THT:R_Axial_DIN0207_L6.3mm_D2.5mm_P10.16mm_Horizontal" H 6400 3800 50  0001 C CNN
 F 3 "~" H 6400 3800 50  0001 C CNN
 	1    6400 3800
@@
 F 0 "R7" V 6195 4050 50  0000 C CNN
 F 1 "220R" V 6286 4050 50  0000 C CNN
-F 2 "Resistor_THT:R_Axial_DIN0207_L6.3mm_D2.5mm_P7.62mm_Horizontal" H 6400 4050 50  0001 C CNN
+F 2 "Resistor_THT:R_Axial_DIN0207_L6.3mm_D2.5mm_P10.16mm_Horizontal" H 6400 4050 50  0001 C CNN
 F 3 "~" H 6400 4050 50  0001 C CNN
 	1    6400 4050
@@
 F 0 "R4" V 4745 7050 50  0000 C CNN
 F 1 "10R3" V 4836 7050 50  0000 C CNN
-F 2 "Resistor_THT:R_Axial_DIN0207_L6.3mm_D2.5mm_P7.62mm_Horizontal" H 4950 7050 50  0001 C CNN
+F 2 "Resistor_THT:R_Axial_DIN0207_L6.3mm_D2.5mm_P10.16mm_Horizontal" H 4950 7050 50  0001 C CNN
 F 3 "~" H 4950 7050 50  0001 C CNN
 	1    4950 7050
@@
 	9300 2100 9300 1650
 Wire Wire Line
-	9300 1650 8550 1650
-Wire Wire Line
 	9450 2400 9550 2400
 Wire Wire Line
 	9300 2300 9300 4500
-Wire Wire Line
-	9300 4500 8500 4500
 Wire Wire Line
 	9300 2300 9550 2300
@@
 Wire Wire Line
 	9050 2100 9050 3150
+Wire Wire Line
+	7750 1650 9300 1650
+Wire Wire Line
+	7750 2700 9200 2700
+Wire Wire Line
+	7700 4500 9300 4500
 $EndSCHEMATC
