File: pcb/StopLight4/StopLight4.kicad_pcb (KiCad board)
At the start: 2 copper layers, 100 x 120.5 mm, 59 parts, among them J1 1935336, J2 1935336, J3 Remote Header, Q1 BT136-600, Q2 BT136-600, Q3 BT136-600, Q5 2N3904, T1 FS20-600, U1 L7805, U10 MOC3021M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

Commit message: update docs and status, add pictures
Other:
- net class ACPower removed
- net class ACSignal removed
- net class DCPower removed
- net class Default removed
- net class PSULow removed
